File: buck.kicad_sch (KiCad schematic)
At the start: 10 parts, among them J3 Water_Pump, J5 694106402002, Q1 FDMS86255, U4 LM2596S-5

Commit message: Added footprints for speakers
And changed size of other pin headers
Parts:
- J3: footprint Connector_PinHeader_1.00mm:PinHeader_1x02_P1.00mm_Vertical_SMD_Pin1Right -> Connector_PinHeader_1.27mm:PinHeader_1x02_P1.27mm_Vertical_SMD_Pin1Left
Changed lines of the file:
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@@
 			)
 		)
-		(property "Footprint" "Connector_PinHeader_1.00mm:PinHeader_1x02_P1.00mm_Vertical_SMD_Pin1Right"
+		(property "Footprint" "Connector_PinHeader_1.27mm:PinHeader_1x02_P1.27mm_Vertical_SMD_Pin1Left"
 			(at 83.82 97.79 0)
 			(effects
