File: tempSensor.kicad_sch (KiCad schematic)
At the start: 5 parts, among them U2 TMP175AIDR

Commit message: Added TMP157 footprint
Fixed and added the rest of footprints to the PCB
Parts:
- U2: footprint TMP175AIDR:SOIC127P599X175-8N -> TMP175AIDR:TMP-SOIC127P599X175-8N
Changed lines of the file:
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@@
 			)
 		)
-		(property "Footprint" "TMP175AIDR:SOIC127P599X175-8N"
+		(property "Footprint" "TMP175AIDR:TMP-SOIC127P599X175-8N"
 			(at 138.43 83.82 0)
 			(effects
