File: codec.kicad_sch (KiCad schematic)
At the start: 24 parts, among them U1 UDA1380HN_N2

Commit message: Finished PCB
Also added GNDA and GNDD references, to be changed back to GND later. Also added wires connecting ground polygons
Connections:
- net GND renamed GNDD
Changed lines of the file:
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@@
 	)
 	(symbol
-		(lib_id "power:GND")
+		(lib_id "power:GNDD")
 		(at 237.49 76.2 0)
 		(unit 1)
@@
 			)
 		)
-		(property "Value" "GND"
-			(at 237.49 80.264 0)
+		(property "Value" "GNDD"
+			(at 237.49 79.375 0)
 			(effects
 				(font
@@
 			)
 		)
-		(property "Description" "Power symbol creates a global label with name \"GND\" , ground"
+		(property "Description" "Power symbol creates a global label with name \"GNDD\" , digital ground"
 			(at 237.49 76.2 0)
 			(effects
@@
 	)
 	(symbol
-		(lib_id "power:GND")
+		(lib_id "power:GNDD")
 		(at 240.03 50.8 0)
 		(unit 1)
@@
 			)
 		)
-		(property "Value" "GND"
-			(at 240.03 54.356 0)
+		(property "Value" "GNDD"
+			(at 240.03 53.975 0)
 			(effects
 				(font
@@
 			)
 		)
-		(property "Description" "Power symbol creates a global label with name \"GND\" , ground"
+		(property "Description" "Power symbol creates a global label with name \"GNDD\" , digital ground"
 			(at 240.03 50.8 0)
 			(effects
@@
 	)
 	(symbol
-		(lib_id "power:GND")
+		(lib_id "power:GNDD")
 		(at 45.72 139.7 0)
 		(mirror y)
@@
 			)
 		)
-		(property "Value" "GND"
-			(at 45.72 144.78 0)
+		(property "Value" "GNDD"
+			(at 45.72 143.51 0)
 			(effects
 				(font
@@
 			)
 		)
-		(property "Description" "Power symbol creates a global label with name \"GND\" , ground"
+		(property "Description" "Power symbol creates a global label with name \"GNDD\" , digital ground"
 			(at 45.72 139.7 0)
 			(effects
@@
 	)
 	(symbol
-		(lib_id "power:GND")
+		(lib_id "power:GNDD")
 		(at 129.54 85.09 0)
 		(unit 1)
@@
 			)
 		)
-		(property "Value" "GND"
-			(at 132.842 86.614 0)
+		(property "Value" "GNDD"
+			(at 129.54 88.265 0)
 			(effects
 				(font
@@
 			)
 		)
-		(property "Description" "Power symbol creates a global label with name \"GND\" , ground"
+		(property "Description" "Power symbol creates a global label with name \"GNDD\" , digital ground"
 			(at 129.54 85.09 0)
 			(effects
@@
 	)
 	(symbol
-		(lib_id "power:GND")
+		(lib_id "power:GNDD")
 		(at 129.54 74.93 0)
 		(unit 1)
@@
 			)
 		)
-		(property "Value" "GND"
-			(at 132.842 76.454 0)
+		(property "Value" "GNDD"
+			(at 129.54 78.105 0)
 			(effects
 				(font
@@
 			)
 		)
-		(property "Description" "Power symbol creates a global label with name \"GND\" , ground"
+		(property "Description" "Power symbol creates a global label with name \"GNDD\" , digital ground"
 			(at 129.54 74.93 0)
 			(effects
@@
 	)
 	(symbol
-		(lib_id "power:GND")
+		(lib_id "power:GNDD")
 		(at 113.03 62.23 0)
 		(unit 1)
@@
 			)
 		)
-		(property "Value" "GND"
-			(at 113.03 67.31 0)
+		(property "Value" "GNDD"
+			(at 113.03 65.405 0)
 			(effects
 				(font
@@
 			)
 		)
-		(property "Description" "Power symbol creates a global label with name \"GND\" , ground"
+		(property "Description" "Power symbol creates a global label with name \"GNDD\" , digital ground"
 			(at 113.03 62.23 0)
 			(effects
@@
 	)
 	(symbol
-		(lib_id "power:GND")
+		(lib_id "power:GNDD")
 		(at 146.05 118.11 0)
 		(unit 1)
@@
 			)
 		)
-		(property "Value" "GND"
-			(at 146.05 121.92 0)
+		(property "Value" "GNDD"
+			(at 146.05 121.285 0)
 			(effects
 				(font
@@
 			)
 		)
-		(property "Description" "Power symbol creates a global label with name \"GND\" , ground"
+		(property "Description" "Power symbol creates a global label with name \"GNDD\" , digital ground"
 			(at 146.05 118.11 0)
 			(effects
@@
 	)
 	(symbol
-		(lib_id "power:GND")
+		(lib_id "power:GNDD")
 		(at 45.72 161.29 0)
 		(mirror y)
@@
 			)
 		)
-		(property "Value" "GND"
-			(at 45.72 166.37 0)
+		(property "Value" "GNDD"
+			(at 45.72 165.1 0)
 			(effects
 				(font
@@
 			)
 		)
-		(property "Description" "Power symbol creates a global label with name \"GND\" , ground"
+		(property "Description" "Power symbol creates a global label with name \"GNDD\" , digital ground"
 			(at 45.72 161.29 0)
 			(effects
@@
 	)
 	(symbol
-		(lib_id "power:GND")
+		(lib_id "power:GNDD")
 		(at 86.36 180.34 0)
 		(unit 1)
@@
 			)
 		)
-		(property "Value" "GND"
-			(at 86.36 185.42 0)
+		(property "Value" "GNDD"
+			(at 86.36 184.15 0)
 			(effects
 				(font
@@
 			)
 		)
-		(property "Description" "Power symbol creates a global label with name \"GND\" , ground"
+		(property "Description" "Power symbol creates a global label with name \"GNDD\" , digital ground"
 			(at 86.36 180.34 0)
 			(effects
@@
 	)
 	(symbol
-		(lib_id "power:GND")
+		(lib_id "power:GNDD")
 		(at 137.16 106.68 0)
 		(unit 1)
@@
 			)
 		)
-		(property "Value" "GND"
-			(at 137.16 110.49 0)
+		(property "Value" "GNDD"
+			(at 137.16 109.855 0)
 			(effects
 				(font
@@
 			)
 		)
-		(property "Description" "Power symbol creates a global label with name \"GND\" , ground"
+		(property "Description" "Power symbol creates a global label with name \"GNDD\" , digital ground"
 			(at 137.16 106.68 0)
 			(effects
@@
 	)
 	(symbol
-		(lib_id "power:GND")
+		(lib_id "power:GNDD")
 		(at 45.72 181.61 0)
 		(mirror y)
@@
 			)
 		)
-		(property "Value" "GND"
-			(at 45.72 186.69 0)
+		(property "Value" "GNDD"
+			(at 45.72 185.42 0)
 			(effects
 				(font
@@
 			)
 		)
-		(property "Description" "Power symbol creates a global label with name \"GND\" , ground"
+		(property "Description" "Power symbol creates a global label with name \"GNDD\" , digital ground"
 			(at 45.72 181.61 0)
 			(effects
@@
 	)
 	(symbol
-		(lib_id "power:GND")
+		(lib_id "power:GNDD")
 		(at 135.89 62.23 0)
 		(unit 1)
@@
 			)
 		)
-		(property "Value" "GND"
-			(at 135.89 66.04 0)
+		(property "Value" "GNDD"
+			(at 135.89 65.405 0)
 			(effects
 				(font
@@
 			)
 		)
-		(property "Description" "Power symbol creates a global label with name \"GND\" , ground"
+		(property "Description" "Power symbol creates a global label with name \"GNDD\" , digital ground"
 			(at 135.89 62.23 0)
 			(effects
@@
 	)
 	(symbol
-		(lib_id "power:GND")
+		(lib_id "power:GNDD")
 		(at 148.59 140.97 0)
 		(unit 1)
@@
 			)
 		)
-		(property "Value" "GND"
-			(at 148.59 146.05 0)
+		(property "Value" "GNDD"
+			(at 148.59 144.145 0)
 			(effects
 				(font
@@
 			)
 		)
-		(property "Description" "Power symbol creates a global label with name \"GND\" , ground"
+		(property "Description" "Power symbol creates a global label with name \"GNDD\" , digital ground"
 			(at 148.59 140.97 0)
 			(effects

Commit message: Made it smaller
Suddenly I had 81 errors??? Now down to 30 from the codec footprint setup
Parts:
- FB1, FB2: footprint OtherComponents:FerriteBead_742861160_0603 -> FerriteBead:FerriteBead_742861160_0603
Changed lines of the file:
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@@
 			)
 		)
-		(property "Footprint" "OtherComponents:FerriteBead_742861160_0603"
+		(property "Footprint" "FerriteBead:FerriteBead_742861160_0603"
 			(at 80.01 156.718 90)
 			(effects
@@
 			)
 		)
-		(property "Footprint" "OtherComponents:FerriteBead_742861160_0603"
+		(property "Footprint" "FerriteBead:FerriteBead_742861160_0603"
 			(at 76.2 164.592 90)
 			(effects

Commit message: Changed grounds and began with new planes
Connections:
- net GNDD renamed GND
